File: KiCad Projects/Embedded_Robot_PCB/Embedded_Robot_PCB.kicad_pcb (KiCad board)
At the start: 2 copper layers, 7 parts, among them U1 STM32F103RCTx

Commit message: 4/24 Inclass Work
Parts:
- added C7: 0.01uF, Capacitor_SMD:C_0805_2012Metric_Pad1.18x1.45mm_HandSolder, F.Cu at (107.0, 100.5)
- added C8: 22pF, Capacitor_SMD:C_0805_2012Metric_Pad1.18x1.45mm_HandSolder, F.Cu at (81.0, 91.3)
- added C9: 22pF, Capacitor_SMD:C_0805_2012Metric_Pad1.18x1.45mm_HandSolder, F.Cu at (81.0, 94.3)
- added D1: USB_PWR_LED, LED_SMD:LED_0805_2012Metric_Pad1.15x1.40mm_HandSolder, F.Cu at (76.5, 90.0)
- added D2: uP_PWR_LED, LED_SMD:LED_0805_2012Metric_Pad1.15x1.40mm_HandSolder, F.Cu at (132.3, 86.6)
- added D3: USER_LED, LED_SMD:LED_0805_2012Metric_Pad1.15x1.40mm_HandSolder, F.Cu at (132.3, 89.6)
- added F1: PTCSMD, Fuse:Fuse_0805_2012Metric_Pad1.15x1.40mm_HandSolder, F.Cu at (66.5, 77.0)
- added J1: USB_B_Mini, Connector_USB:USB_Mini-B_Lumberg_2486_01_Horizontal, F.Cu at (75.4, 81.6)
- added R1: 10k, Resistor_SMD:R_0805_2012Metric_Pad1.20x1.40mm_HandSolder, F.Cu at (117.5, 100.5)
- added R2: 22, Resistor_SMD:R_0805_2012Metric_Pad1.20x1.40mm_HandSolder, F.Cu at (66.5, 81.3)
- added R3: 22, Resistor_SMD:R_0805_2012Metric_Pad1.20x1.40mm_HandSolder, F.Cu at (66.5, 84.3)
- added R4: 10k, Resistor_SMD:R_0805_2012Metric_Pad1.20x1.40mm_HandSolder, F.Cu at (66.5, 87.2)
- added R5: 10k, Resistor_SMD:R_0805_2012Metric_Pad1.20x1.40mm_HandSolder, F.Cu at (137.0, 86.5)
- added R6: 10k, Resistor_SMD:R_0805_2012Metric_Pad1.20x1.40mm_HandSolder, F.Cu at (137.0, 89.5)
- added S1: SW_uP_Boot, SW_uP_Boot:SW_JS202011SCQN, F.Cu at (99.3, 103.8)
- added SW1: SW_uP_Reset, SW_uP_Reset:SW_uP_Reset, F.Cu at (100.6, 95.7)
- added U2: USBLC6-2SC6, Package_TO_SOT_SMD:SOT-23-6, F.Cu at (71.5, 90.9)
- added Y1: Crystal_GND23, Crystal:Crystal_SMD_Abracon_ABM8G-4Pin_3.2x2.5mm, F.Cu at (88.1, 98.2)
- added Y2: 16MHz, Crystal:Crystal_SMD_Abracon_ABM8G-4Pin_3.2x2.5mm, F.Cu at (86.0, 92.0)
Connections:
- U1 pad 44: unconnected-(U1-PA11-Pad44) -> /USB_D-
- U1 pad 45: unconnected-(U1-PA12-Pad45) -> /USB_D+
- U1 pad 5: unconnected-(U1-PD0-Pad5) -> /OSC_IN
- U1 pad 6: unconnected-(U1-PD1-Pad6) -> /OSC_OUT
- U1 pad 60: unconnected-(U1-BOOT0-Pad60) -> /BOOT
- U1 pad 7: unconnected-(U1-NRST-Pad7) -> /RESET

Commit message: Routing
Parts:
- added D4: uP_PWR_LED, LED_SMD:LED_0805_2012Metric_Pad1.15x1.40mm_HandSolder, F.Cu at (103.0, 63.0)
- added J2: CONN_MPU6050, Connector_PinSocket_2.54mm:PinSocket_1x08_P2.54mm_Vertical, F.Cu at (91.5, 51.2)
- added J3: CONN_ULTRA, Connector_PinSocket_2.54mm:PinSocket_1x04_P2.54mm_Vertical, F.Cu at (134.0, 20.9)
- added MDBT42T-AT1: MDBT42T-AT, MDBT42T-AT:MDBT42T, F.Cu at (114.0, 54.5)
- added R7: 10k, Resistor_SMD:R_0805_2012Metric_Pad1.20x1.40mm_HandSolder, F.Cu at (103.0, 66.0)
- D2: value uP_PWR_LED -> BL_IND_LED
Connections:
- R5 pad 1: +3V3 -> Net-(MDBT42T-AT1-INDICATOR)
