File: KiCad Projects/Embedded_Robot_PCB/Embedded_Robot_PCB.kicad_sch (KiCad schematic)
At the start: 7 parts, among them U1 STM32F103RCTx

Commit message: 4/24 Inclass Work
Parts:
- added C7: 0.01uF, Capacitor_SMD:C_0805_2012Metric_Pad1.18x1.45mm_HandSolder, symbol Device:C_Small
- added C8, C9: 22pF, Capacitor_SMD:C_0805_2012Metric_Pad1.18x1.45mm_HandSolder, symbol Device:C_Small
- added D1: USB_PWR_LED, LED_SMD:LED_0805_2012Metric_Pad1.15x1.40mm_HandSolder, symbol Device:LED_Small
- added D2: uP_PWR_LED, LED_SMD:LED_0805_2012Metric_Pad1.15x1.40mm_HandSolder, symbol Device:LED_Small
- added D3: USER_LED, LED_SMD:LED_0805_2012Metric_Pad1.15x1.40mm_HandSolder, symbol Device:LED_Small
- added F1: PTCSMD, Fuse:Fuse_0805_2012Metric_Pad1.15x1.40mm_HandSolder, symbol Device:Polyfuse_Small
- added J1: USB_B_Mini, Connector_USB:USB_Mini-B_Lumberg_2486_01_Horizontal, symbol Connector:USB_B_Mini
- added R1, R4, R5, R6: 10k, Resistor_SMD:R_0805_2012Metric_Pad1.20x1.40mm_HandSolder, symbol Device:R_Small
- added R2, R3: 22, Resistor_SMD:R_0805_2012Metric_Pad1.20x1.40mm_HandSolder, symbol Device:R_Small
- added S1: SW_uP_Boot, SW_uP_Boot:SW_JS202011SCQN, symbol SW_uP_Boot:JS202011SCQN
- added SW1: SW_uP_Reset, SW_uP_Reset:SW_uP_Reset, symbol Switch:SW_SPST
- added U2: USBLC6-2SC6, Package_TO_SOT_SMD:SOT-23-6, symbol Power_Protection:USBLC6-2SC6
- added Y2: 16MHz, Crystal:Crystal_SMD_Abracon_ABM8G-4Pin_3.2x2.5mm, symbol Device:Crystal_GND24
Connections:
- net +3V3: now also R5.1, S1.1
- net GND: now also C7.1, C8.1, C9.1, D1.1 (K), D2.1 (K), D3.1 (K), J1.5 (GND), S1.3, SW1.1 (A), U2.2 (GND), Y2.2, Y2.4
- net USB_D-: now reaches U1.44 (PA11)
- net USB_D-: now also U2.6 (I/O1)
- net USB_D+: now reaches U1.45 (PA12)
- net USB_D+: now also U2.4 (I/O2)
- net OSC_IN: now reaches U1.5 (PD0)
- net OSC_IN: now also C9.2, Y2.1
- net OSC_OUT: now reaches U1.6 (PD1)
- net OSC_OUT: now also C8.2, Y2.3
- net BOOT: now reaches U1.60 (BOOT0)
- net BOOT: now also R1.1
- net RESET: now reaches U1.7 (NRST)
- net RESET: now also C7.2, SW1.2 (B)
- new net: D2.2 (A), R5.2
- new net: F1.2, J1.1 (VBUS)
- new net: R1.2, S1.2
- new net: D3.2 (A), R6.2
- new net: D1.2 (A), R4.2
- new net D+: J1.3 (D+), R3.1
- new net D-: J1.2 (D-), R2.1
- new net USB_CONN_D+: R3.2, U2.3 (I/O2)
- new net USB_CONN_D-: R2.2, U2.1 (I/O1)
- new net USER_LED: R6.1
- new net Vusb: F1.1, R4.1, U2.5 (VBUS)
- no-connect marks 1 -> 6
Other:
- note added: "Decoupling Caps"
- note added: "Microcontroller"
- moved on the sheet: C1, C2, C3, C4, C5, C6, U1

Commit message: Routing
Parts:
- added C10, C11: 0.1uF, Capacitor_SMD:C_0805_2012Metric_Pad1.18x1.45mm_HandSolder, symbol Device:C_Small
- added D4: uP_PWR_LED, LED_SMD:LED_0805_2012Metric_Pad1.15x1.40mm_HandSolder, symbol Device:LED_Small
- added J2: CONN_MPU6050, Connector_PinSocket_2.54mm:PinSocket_1x08_P2.54mm_Vertical, symbol Connector_Generic:Conn_01x08
- added J3: CONN_ULTRA, Connector_PinSocket_2.54mm:PinSocket_1x04_P2.54mm_Vertical, symbol Connector_Generic:Conn_01x04
- added J4: CONN_SWD, symbol Connector_Generic:Conn_01x04
- added J5: CONN_5V, Connector_JST:JST_XH_B2B-XH-A_1x02_P2.50mm_Vertical, symbol Connector_Generic:Conn_01x02
- added J6: CONN_3V3, Connector_JST:JST_XH_B2B-XH-A_1x02_P2.50mm_Vertical, symbol Connector_Generic:Conn_01x02
- added J7: CONN_DRIVE, symbol Connector_Generic:Conn_01x04
- added J8: CONN_HALL, symbol Connector_Generic:Conn_01x05
- added LED1, LED2: IN-PI55TATPRPGPB, RGB_LED:INPI55TATPRPGPB, symbol RGB_LED:IN-PI55TATPRPGPB
- added MDBT42T-AT1: MDBT42T-AT, MDBT42T-AT:MDBT42T, symbol MDBT42T-AT:MDBT42T-AT
- added Q1: BSS138, Package_TO_SOT_SMD:SOT-23, symbol Transistor_FET:BSS138
- added R10, R7, R8, R9: 10k, Resistor_SMD:R_0805_2012Metric_Pad1.20x1.40mm_HandSolder, symbol Device:R_Small
- added SW2: SW_USER, SW_uP_Reset:SW_uP_Reset, symbol Switch:SW_SPST
- D2: value uP_PWR_LED -> BL_IND_LED
Connections:
- net +3V3: now also J4.4 (Pin_4), J6.1 (Pin_1), MDBT42T-AT1.15 (VDD), Q1.1 (G), R7.1, R8.1, R9.1; no longer R5.1
- net GND: now also C10.2, C11.2, D4.1 (K), J2.2 (Pin_2), J3.1 (Pin_1), J4.2 (Pin_2), J5.2 (Pin_2), J6.2 (Pin_2), LED1.3 (VSS), LED2.3 (VSS), MDBT42T-AT1.1 (GND@1), MDBT42T-AT1.10 (GND@10), MDBT42T-AT1.12 (FLASH_DEFAULT), MDBT42T-AT1.16 (GND@16), MDBT42T-AT1.19 (GND@19), MDBT42T-AT1.9 (UART_PD), SW2.2 (B)
- net USER_LED: now also U1.2 (PC13)
- net IMU_INT: now reaches U1.57 (PB5)
- net IMU_INT: now also J2.8 (Pin_8)
- net IMU_I2C_SCL: now reaches U1.58 (PB6)
- net IMU_I2C_SCL: now also J2.3 (Pin_3)
- net IMU_I2C_SDA: now reaches U1.59 (PB7)
- net IMU_I2C_SDA: now also J2.4 (Pin_4)
- new net: MDBT42T-AT1.5 (INDICATOR), R5.1
- new net: D4.2 (A), R7.2
- new net: LED1.2 (DOUT), LED2.4 (DIN)
- new net: LED1.4 (DIN), Q1.2 (S), R10.2
- new net +5V: C10.1, C11.1, J2.1 (Pin_1), J3.4 (Pin_4), J5.1 (Pin_1), LED1.1 (VDD), LED2.1 (VDD), R10.1
- new net BL_RX: MDBT42T-AT1.8 (RX)
- new net BL_TX: MDBT42T-AT1.7 (TX)
- new net BL_WAKEUP: MDBT42T-AT1.6 (WAKEUP)
- new net RGB_DIN: Q1.3 (D), R9.2
- new net SWDCLK: J4.3 (Pin_3)
- new net SWDIO: J4.1 (Pin_1)
- new net ULTRA_ECHO: J3.2 (Pin_2)
- new net ULTRA_TRIG: J3.3 (Pin_3)
- new net USER_BUTTON: R8.2, SW2.1 (A)
- no-connect marks 6 -> 18
Other:
- note added: "BLUETOOTH"
- note added: "BUTTON"
- note added: "IMU (MPU6050)"
- note added: "PWR CONN"
- note added: "RBG LED"
- note added: "SWD"
- note added: "ULTRASONIC SENSOR"
- moved on the sheet: D2, R5
